File: funcdec_modB.hw/funcdec_uni.hw.sch (KiCad schematic (older format))
At the start: 27 parts, among them J1 Track2, J2 Track1, J3 PROG, J4 Functions, Q1 BSS138, Q2 AP2626, Q3 AP2626, Q4 AP2626, U1 AP2204K-5.0, U2 ATtiny1614-SS

Commit message: ack circuit correction
Parts:
- removed Q1: BSS138, NGS Elements SMD:SOT23_HS, symbol Device:Q_NMOS_GSD
- added Q1: BC847, NGS Elements SMD:SOT23_HS, symbol Device:Q_NPN_BEC
- R2: value 82R -> 150R
- R3: value 22k -> 15k
- R4: value 100R -> 10k
Connections:
- net GND: now also Q1.2 (E)
- net at R2.2: now also Q1.3 (C)
- net at R4.1: now also Q1.1 (B)
Changed lines of the file:
@@
 P 2550 2700
 F 0 "R2" V 2450 2650 50  0000 L CNN
-F 1 "82R" V 2650 2650 50  0000 L CNN
+F 1 "150R" V 2650 2600 50  0000 L CNN
 F 2 "NGS Elements SMD:SMD_1206_HS" V 2480 2700 50  0001 C CNN
 F 3 "~" H 2550 2700 50  0001 C CNN
@@
 P 2600 3950
 F 0 "R3" V 2500 3900 50  0000 L CNN
-F 1 "22k" V 2700 3900 50  0000 L CNN
+F 1 "15k" V 2700 3900 50  0000 L CNN
 F 2 "NGS Elements SMD:SMD_0805_HS" V 2530 3950 50  0001 C CNN
 F 3 "~" H 2600 3950 50  0001 C CNN
@@
 Connection ~ 1400 3300
 $Comp
-L Device:Q_NMOS_GSD Q1
-U 1 1 5E9BCE6F
-P 2650 3150
-F 0 "Q1" H 2855 3196 50  0000 L CNN
-F 1 "BSS138" H 2855 3105 50  0000 L CNN
-F 2 "NGS Elements SMD:SOT23_HS" H 2850 3250 50  0001 C CNN
-F 3 "~" H 2650 3150 50  0001 C CNN
-	1    2650 3150
-	-1   0    0    -1
-$EndComp
-$Comp
 L power:GND #PWR06
 U 1 1 5E9C2454
@@
 P 2950 3500
 F 0 "R4" H 3020 3546 50  0000 L CNN
-F 1 "100R" H 3020 3455 50  0000 L CNN
+F 1 "10k" H 3020 3455 50  0000 L CNN
 F 2 "NGS Elements SMD:SMD_0805_HS" V 2880 3500 50  0001 C CNN
 F 3 "~" H 2950 3500 50  0001 C CNN
@@
 Wire Wire Line
 	5050 5700 4850 5700
+$Comp
+L Device:Q_NPN_BEC Q1
+U 1 1 5EC2F346
+P 2650 3150
+F 0 "Q1" H 2841 3196 50  0000 L CNN
+F 1 "BC847" H 2841 3105 50  0000 L CNN
+F 2 "NGS Elements SMD:SOT23_HS" H 2850 3250 50  0001 C CNN
+F 3 "~" H 2650 3150 50  0001 C CNN
+	1    2650 3150
+	-1   0    0    -1
+$EndComp
 $EndSCHEMATC

Commit message: corrections and file rename for manf
Parts:
- removed J3: PROG, NGS_Connectors_SMD:Array_1-27mm_1X3_SMD, symbol Connector_Generic:Conn_01x03
- removed Q1: BC847, NGS Elements SMD:SOT23_HS, symbol Device:Q_NPN_BEC
- added J3: Pad1.27x5, NGS_Connectors_SMD:Array_1-27mm_1X5_SMD, symbol Connector_Generic:Conn_01x05
- added Q1: BC817UE, NGS Elements SMD:SOT23-6_HS, symbol Transistor_BJT:BC846BPDW1
- C1: value 10u -> 4.7u
- C2: value 22u -> 10u
- J1: value Track2 -> Padx1
- J2: value Track1 -> Padx1
- J4: value Functions -> Pad1.5x7
- R2: value 150R -> 8R2; footprint NGS Elements SMD:SMD_1206_HS -> NGS Elements SMD:SMD_0805_HS
Connections:
- net ACK: now also U2.6 (PB3); no longer U2.4 (PA6)
- net DCC: now also U2.4 (PA6); no longer U2.11 (PA1)
- net GND: now also C3.1, R2.2, J3.2 (Pin_2), Q1.1 (E1); no longer C3.2
- net VCC: now also C3.2, J3.1 (Pin_1); no longer C3.1
- net at D1.1 (K), D2.1 (K), J4.1 (Pin_1)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: now also Q1.3 (C2); no longer R2.1
- net at U2.10 (~RESET~/PA0): now also J3.3 (Pin_3)
- net at U2.12 (PA2): now also J3.5 (Pin_5)
- net at R4.1: now also Q1.5 (B2), Q1.6 (C1)
- new net: Q1.2 (B1), Q1.4 (E2), R2.1
- new net: J3.4 (Pin_4), U2.11 (PA1)
Other:
- note added: "+U"
- note added: "..."
- note added: "F1"
- note added: "F6"
- note added: "FUNCTIONS"
- note added: "Ou1"
- note added: "Ou2"
- note added: "PROG"
- note added: "Track1"
- note added: "Track2"
- moved on the sheet: C3, R1, R2, R4
